File: alt-panel/alt-panel.kicad_pcb (KiCad board)
At the start: 2 copper layers, 70.8 x 128.5 mm, 23 parts

Commit message: Panel tweak
Parts:
- moved REF** 0.75 mm to (22.5, 94.2)
- moved REF** 0.75 mm to (22.5, 52.2)
- moved REF** 0.31 mm to (30.1, 126.4)
- moved REF** 0.31 mm to (38.3, 126.4)
- moved REF** 0.31 mm to (34.3, 126.4)
- moved REF** 0.31 mm to (26.1, 126.4)
- moved REF** 0.31 mm to (42.1, 126.4)
Changed lines of the file:
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@@
   (net 0 "")
   (footprint "diy-nabra:Vol" (layer "F.Cu")
-    (at 22.5 93.5)
+    (at 22.5 94.25)
     (attr through_hole)
     (fp_text reference "REF**" (at 0 -0.5 unlocked) (layer "F.SilkS") hide
@@
       (effects (font (size 1 1) (thickness 0.15)))
     )
-    (fp_line (start -4.9 1.75) (end 3.7 1.75) (layer "F.SilkS") (width 0.5))
-    (fp_line (start 3.7 1.75) (end 3.7 -2.35) (layer "F.SilkS") (width 0.5))
-    (fp_line (start 3.7 -2.35) (end -5 1.75) (layer "F.SilkS") (width 0.5))
+    (fp_line (start -4.5 1.25) (end 3.5 1.25) (layer "F.SilkS") (width 0.5))
+    (fp_line (start 3.5 -2.85) (end -4.5 1.25) (layer "F.SilkS") (width 0.5))
+    (fp_line (start 3.5 1.25) (end 3.5 -2.85) (layer "F.SilkS") (width 0.5))
   )
   (footprint "diy-nabra:Star" (layer "F.Cu")
@@
   )
   (footprint "diy-nabra:R" (layer "F.Cu")
-    (at 42.0625 126.75)
+    (at 42.0625 126.4375)
     (attr through_hole)
     (fp_text reference "REF**" (at 0 -0.5 unlocked) (layer "F.SilkS") hide
@@
   )
   (footprint "diy-nabra:U" (layer "F.Cu")
-    (at 30.0625 126.75)
+    (at 30.0625 126.4375)
     (attr through_hole)
     (fp_text reference "REF**" (at 0 -0.5 unlocked) (layer "F.SilkS") hide
@@
   )
   (footprint "diy-nabra:E" (layer "F.Cu")
-    (at 38.3125 126.75)
+    (at 38.3125 126.4375)
     (attr through_hole)
     (fp_text reference "REF**" (at 0 -0.5 unlocked) (layer "F.SilkS") hide
@@
   )
   (footprint "diy-nabra:Vol" (layer "F.Cu")
-    (at 22.5 51.5)
+    (at 22.5 52.25)
     (attr through_hole)
     (fp_text reference "REF**" (at 0 -0.5 unlocked) (layer "F.SilkS") hide
@@
       (effects (font (size 1 1) (thickness 0.15)))
     )
-    (fp_line (start 3.7 1.75) (end 3.7 -2.35) (layer "F.SilkS") (width 0.5))
-    (fp_line (start 3.7 -2.35) (end -5 1.75) (layer "F.SilkS") (width 0.5))
-    (fp_line (start -4.9 1.75) (end 3.7 1.75) (layer "F.SilkS") (width 0.5))
+    (fp_line (start 3.5 1.25) (end 3.5 -2.85) (layer "F.SilkS") (width 0.5))
+    (fp_line (start 3.5 -2.85) (end -4.5 1.25) (layer "F.SilkS") (width 0.5))
+    (fp_line (start -4.5 1.25) (end 3.5 1.25) (layer "F.SilkS") (width 0.5))
   )
   (footprint "diy-nabra:Freq" (layer "F.Cu")
@@
   )
   (footprint "diy-nabra:B" (layer "F.Cu")
-    (at 34.3125 126.75)
+    (at 34.3125 126.4375)
     (attr through_hole)
     (fp_text reference "REF**" (at 0 -0.5 unlocked) (layer "F.SilkS") hide
@@
   )
   (footprint "diy-nabra:D" (layer "F.Cu")
-    (at 26.0625 126.75)
+    (at 26.0625 126.4375)
     (attr through_hole)
     (fp_text reference "REF**" (at 0 -0.5 unlocked) (layer "F.SilkS") hide
@@
     (style (thickness 0.15) (arrow_length 1.27) (text_position_mode 0) (extension_height 0.58642) (extension_offset 0.5) keep_text_aligned)
   )
+  (dimension (type aligned) (layer "User.5")
+    (pts (xy 26.0625 126.4375) (xy 26.0625 128.5))
+    (height 2.0625)
+    (gr_text "2.0625 mm" (at 22.85 127.46875 90) (layer "User.5")
+      (effects (font (size 1 1) (thickness 0.15)))
+    )
+    (format (units 3) (units_format 1) (precision 4))
+    (style (thickness 0.1) (arrow_length 1.27) (text_position_mode 0) (extension_height 0.58642) (extension_offset 0.5) keep_text_aligned)
+  )
+  (group "" (id 0d563b23-814b-4728-b3a5-325349d469fb)
+    (members
+      83bbdb87-3dc1-40f5-bf5e-3bb0f8dfc548
+      9182484b-068e-4ce4-bc1c-fd9c0d48bc42
+      91dda16f-f6ba-47f8-b9ff-bca5dbff204d
+      9e539c59-6346-4901-bd6a-7dc90968b8dc
+      d751be33-bc96-4cde-8cd7-54ee5cf97ea0
+    )
+  )
   (group "" (id df2dbb8d-2e52-479c-9aa7-c540bfef44bb)

Commit message: Panel tweaks
Parts:
- moved REF** 0.25 mm to (6.50, 42.6)
- moved REF** 0.25 mm to (6.50, 84.7)
Other:
- outline, holes or cut-outs redrawn

Commit message: nologo panel and branch
Parts:
- removed the REF** at (30.1, 126.4)
- removed the REF** at (38.3, 126.4)
- removed the REF** at (34.3, 126.4)
- removed the REF** at (26.1, 126.4)
- removed the REF** at (42.1, 126.4)
Changed lines of the file:
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@@
     (fp_line (start -2.45 2.4) (end 2.55 2.4) (layer "F.SilkS") (width 0.35))
-  )
-  (footprint "diy-nabra:R" (layer "F.Cu")
-    (at 42.0625 126.4375)
-    (attr through_hole)
-    (fp_text reference "REF**" (at 0 -0.5 unlocked) (layer "F.SilkS") hide
-      (effects (font (size 1 1) (thickness 0.15)))
-    )
-    (fp_text value "R" (at 0 1 unlocked) (layer "F.Fab") hide
-      (effects (font (size 1 1) (thickness 0.15)))
-    )
-    (fp_line (start 0.5 -2.5) (end 2.5 0) (layer "F.SilkS") (width 0.25))
-    (fp_line (start 2.5 -3) (end 2 -2.5) (layer "F.SilkS") (width 0.25))
-    (fp_line (start 2.5 -4.5) (end 2.5 -3) (layer "F.SilkS") (width 0.25))
-    (fp_line (start 0 -5) (end 2 -5) (layer "F.SilkS") (width 0.25))
-    (fp_line (start 2 -5) (end 2.5 -4.5) (layer "F.SilkS") (width 0.25))
-    (fp_line (start 2 -2.5) (end 0.5 -2.5) (layer "F.SilkS") (width 0.25))
-    (fp_line (start 0 -5) (end 0 0) (layer "F.SilkS") (width 0.25))
   )
   (footprint "diy-nabra:Star" (layer "F.Cu")
@@
     (fp_line (start 2.5 -0.5) (end 2.5 -2) (layer "F.SilkS") (width 0.25))
   )
-  (footprint "diy-nabra:U" (layer "F.Cu")
-    (at 30.0625 126.4375)
-    (attr through_hole)
-    (fp_text reference "REF**" (at 0 -0.5 unlocked) (layer "F.SilkS") hide
-      (effects (font (size 1 1) (thickness 0.15)))
-    )
-    (fp_text value "U" (at 0 1 unlocked) (layer "F.Fab") hide
-      (effects (font (size 1 1) (thickness 0.15)))
-    )
-    (fp_text user "${REFERENCE}" (at 0 2.5 unlocked) (layer "F.Fab") hide
-      (effects (font (size 1 1) (thickness 0.15)))
-    )
-    (fp_line (start 2.5 0) (end 1 0) (layer "F.SilkS") (width 0.25))
-    (fp_line (start 1 0) (end 0 -1) (layer "F.SilkS") (width 0.25))
-    (fp_line (start 2.5 -5) (end 2.5 0) (layer "F.SilkS") (width 0.25))
-    (fp_line (start 0 -5) (end 0 -1) (layer "F.SilkS") (width 0.25))
-  )
-  (footprint "diy-nabra:E" (layer "F.Cu")
-    (at 38.3125 126.4375)
-    (attr through_hole)
-    (fp_text reference "REF**" (at 0 -0.5 unlocked) (layer "F.SilkS") hide
-      (effects (font (size 1 1) (thickness 0.15)))
-    )
-    (fp_text value "E" (at 0 1 unlocked) (layer "F.Fab") hide
-      (effects (font (size 1 1) (thickness 0.15)))
-    )
-    (fp_text user "${REFERENCE}" (at 0 2.5 unlocked) (layer "F.Fab") hide
-      (effects (font (size 1 1) (thickness 0.15)))
-    )
-    (fp_line (start 0 -5) (end 0 0) (layer "F.SilkS") (width 0.25))
-    (fp_line (start 2 0) (end 2.5 0) (layer "F.SilkS") (width 0.25))
-    (fp_line (start 0 -5) (end 2 -5) (layer "F.SilkS") (width 0.25))
-    (fp_line (start 2 -2.5) (end 0 -2.5) (layer "F.SilkS") (width 0.25))
-    (fp_line (start 0 0) (end 2 0) (layer "F.SilkS") (width 0.25))
-    (fp_line (start 2 -5) (end 2.5 -5) (layer "F.SilkS") (width 0.25))
-  )
   (footprint "diy-nabra:Vol" (layer "F.Cu")
     (at 22.5 52.25)
@@
     (fp_line (start -1 2.125) (end -4 0.0125) (layer "F.SilkS") (width 0.5))
     (fp_line (start 1 -2.375) (end 4 0) (layer "F.SilkS") (width 0.5))
-  )
-  (footprint "diy-nabra:B" (layer "F.Cu")
-    (at 34.3125 126.4375)
-    (attr through_hole)
-    (fp_text reference "REF**" (at 0 -0.5 unlocked) (layer "F.SilkS") hide
-      (effects (font (size 1 1) (thickness 0.15)))
-    )
-    (fp_text value "B" (at 0 1 unlocked) (layer "F.Fab") hide
-      (effects (font (size 1 1) (thickness 0.15)))
-    )
-    (fp_line (start 2 -2.5) (end 0.5 -2.5) (layer "F.SilkS") (width 0.25))
-    (fp_line (start 0 -5) (end 2 -5) (layer "F.SilkS") (width 0.25))
-    (fp_line (start 2 0) (end 2.5 -0.5) (layer "F.SilkS") (width 0.25))
-    (fp_line (start 2 -5) (end 2.5 -4.5) (layer "F.SilkS") (width 0.25))
-    (fp_line (start 0 -5) (end 0 0) (layer "F.SilkS") (width 0.25))
-    (fp_line (start 2.5 -4.5) (end 2.5 -3) (layer "F.SilkS") (width 0.25))
-    (fp_line (start 2.5 -0.5) (end 2.5 -2) (layer "F.SilkS") (width 0.25))
-    (fp_line (start 2.5 -3) (end 2 -2.5) (layer "F.SilkS") (width 0.25))
-    (fp_line (start 2.5 -2) (end 2 -2.5) (layer "F.SilkS") (width 0.25))
-    (fp_line (start 0 0) (end 2 0) (layer "F.SilkS") (width 0.25))
   )
   (footprint "diy-nabra:A" (layer "F.Cu")
@@
     (fp_line (start 3.8125 -2.5625) (end 0.5625 -2.5625) (layer "F.SilkS") (width 0.25))
     (fp_line (start 3.0625 -0.0625) (end 3.8125 -0.0625) (layer "F.SilkS") (width 0.25))
-  )
-  (footprint "diy-nabra:D" (layer "F.Cu")
-    (at 26.0625 126.4375)
-    (attr through_hole)
-    (fp_text reference "REF**" (at 0 -0.5 unlocked) (layer "F.SilkS") hide
-      (effects (font (size 1 1) (thickness 0.15)))
-    )
-    (fp_text value "D" (at 0 1 unlocked) (layer "F.Fab") hide
-      (effects (font (size 1 1) (thickness 0.15)))
-    )
-    (fp_text user "${REFERENCE}" (at 0 2.5 unlocked) (layer "F.Fab") hide
-      (effects (font (size 1 1) (thickness 0.15)))
-    )
-    (fp_line (start 1.5 -5) (end 2.5 -4) (layer "F.SilkS") (width 0.25))
-    (fp_line (start 0 -5) (end 1.5 -5) (layer "F.SilkS") (width 0.25))
-    (fp_line (start 2.5 -4) (end 2.5 -1) (layer "F.SilkS") (width 0.25))
-    (fp_line (start 1.5 0) (end 2.5 -1) (layer "F.SilkS") (width 0.25))
-    (fp_line (start 0 -5) (end 0 0) (layer "F.SilkS") (width 0.25))
-    (fp_line (start 0 0) (end 1.5 0) (layer "F.SilkS") (width 0.25))
   )
   (footprint "diy-nabra:QRes" (layer "F.Cu")
@@
     (style (thickness 0.15) (arrow_length 1.27) (text_position_mode 0) (extension_height 0.58642) (extension_offset 0.5) keep_text_aligned)
   )
-  (dimension (type aligned) (layer "User.5")
-    (pts (xy 26.0625 126.4375) (xy 26.0625 128.5))
-    (height 2.0625)
-    (gr_text "2.0625 mm" (at 22.85 127.46875 90) (layer "User.5")
-      (effects (font (size 1 1) (thickness 0.15)))
-    )
-    (format (units 3) (units_format 1) (precision 4))
-    (style (thickness 0.1) (arrow_length 1.27) (text_position_mode 0) (extension_height 0.58642) (extension_offset 0.5) keep_text_aligned)
-  )
-  (group "" (id 0d563b23-814b-4728-b3a5-325349d469fb)
-    (members
-      83bbdb87-3dc1-40f5-bf5e-3bb0f8dfc548
-      9182484b-068e-4ce4-bc1c-fd9c0d48bc42
-      91dda16f-f6ba-47f8-b9ff-bca5dbff204d
-      9e539c59-6346-4901-bd6a-7dc90968b8dc
-      d751be33-bc96-4cde-8cd7-54ee5cf97ea0
-    )
-  )
   (group "" (id 641ec3e6-cd5f-4009-b963-b6bfa61a5a5c)
